File: crowd chase el.sch (EAGLE design)
At the start: 27 parts, among them IC2 PIC18F1220P, U4 TRIAC

Commit message: No more airwires
Parts:
- removed C3: 10uF, SparkFun:CAP_POL1206
- removed U$7: 12MMTACT_MJTP1212, chasetron:12MMTACT_MJTP1212
- added C5, C6: 1uF, rcl:C-US025-025X050
- added IC1: 7805L, linear:7805L
Connections:
- new net DEVICE_MAX_SET: IC2.INT2/P1B/RB2, U$6.P$2
- new net MAX_LED: IC2.RA0/AN0, LED2.A
- new net N$4: BAT1.-, C6.1, IC1.VI
- new net N$8: IC2.INT1/CK/TX/AN5/RB1
- new net NUM_LED: IC2.RA1/AN1/LVDIN, LED1.A
- net DEVICE_NUM_SET: now also IC2.INT0/AN4/RB0
- net EL_C: now also IC2.RA4/T0CKI
- net GND: now also C5.2, C6.2, IC1.GND, R1.2, R2.1, U$6.P$1; no longer C3.-
- net VDD: now also C5.1, IC1.VO, JP3.1; no longer BAT1.-, C3.+
Other:
- moved on the sheet: BAT1, JP3
Changed lines of the file:
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@@
 <part name="C2" library="SparkFun" deviceset="CAP" device="PTH2" value="0.1uF"/>
 <part name="GND11" library="supply1" deviceset="GND" device=""/>
-<part name="C3" library="SparkFun" deviceset="CAP_POL" device="1206" value="10uF"/>
-<part name="GND10" library="SparkFun" deviceset="GND" device=""/>
 <part name="GND14" library="SparkFun" deviceset="GND" device=""/>
 <part name="U$2" library="SparkFun" deviceset="FIDUCIAL" device="1X2"/>
@@
 <part name="U$4" library="chasetron" deviceset="12MMTACT_MJTP1212" device=""/>
 <part name="U$6" library="chasetron" deviceset="12MMTACT_MJTP1212" device=""/>
-<part name="U$7" library="chasetron" deviceset="12MMTACT_MJTP1212" device=""/>
 <part name="GND2" library="supply1" deviceset="GND" device=""/>
 <part name="VDD1" library="supply1" deviceset="VDD" device=""/>
@@
 <part name="GND4" library="supply1" deviceset="GND" device=""/>
 <part name="R3" library="rcl" deviceset="R-US_" device="0204/5"/>
+<part name="GND5" library="supply1" deviceset="GND" device=""/>
+<part name="C5" library="rcl" deviceset="C-US" device="025-025X050" value="1uF"/>
+<part name="C6" library="rcl" deviceset="C-US" device="025-025X050" value="1uF"/>
+<part name="IC1" library="linear" deviceset="78*" device="L" technology="05"/>
+<part name="GND6" library="supply1" deviceset="GND" device=""/>
+<part name="GND7" library="supply1" deviceset="GND" device=""/>
 </parts>
 <sheets>
@@
 <instance part="C2" gate="G$1" x="210.82" y="162.56"/>
 <instance part="GND11" gate="1" x="210.82" y="154.94"/>
-<instance part="C3" gate="G$1" x="220.98" y="165.1"/>
-<instance part="GND10" gate="1" x="220.98" y="154.94"/>
 <instance part="GND14" gate="1" x="116.84" y="104.14"/>
 <instance part="U$2" gate="G$1" x="167.64" y="27.94"/>
@@
 <instance part="R1" gate="G$1" x="175.26" y="81.28" rot="R270"/>
 <instance part="R2" gate="G$1" x="185.42" y="81.28" rot="R90"/>
-<instance part="BAT1" gate="G$1" x="187.96" y="175.26"/>
-<instance part="JP3" gate="G$1" x="198.12" y="165.1" rot="R90"/>
+<instance part="BAT1" gate="G$1" x="142.24" y="175.26"/>
+<instance part="JP3" gate="G$1" x="198.12" y="162.56" rot="R270"/>
 <instance part="JP4" gate="G$1" x="93.98" y="170.18"/>
 <instance part="IC2" gate="G$1" x="149.86" y="124.46"/>
 <instance part="U$4" gate="G$1" x="27.94" y="106.68" rot="R270"/>
 <instance part="U$6" gate="G$1" x="22.86" y="50.8"/>
-<instance part="U$7" gate="G$1" x="27.94" y="22.86"/>
-<instance part="GND2" gate="1" x="180.34" y="172.72"/>
+<instance part="GND2" gate="1" x="137.16" y="162.56"/>
 <instance part="VDD1" gate="G$1" x="236.22" y="175.26" rot="R270"/>
 <instance part="Q1" gate="G$1" x="114.3" y="132.08" rot="R90"/>
@@
 <instance part="GND4" gate="1" x="99.06" y="124.46"/>
 <instance part="R3" gate="G$1" x="53.34" y="132.08"/>
+<instance part="GND5" gate="1" x="12.7" y="48.26"/>
+<instance part="C5" gate="G$1" x="180.34" y="172.72"/>
+<instance part="C6" gate="G$1" x="149.86" y="172.72"/>
+<instance part="IC1" gate="A1" x="165.1" y="175.26"/>
+<instance part="GND6" gate="1" x="175.26" y="71.12"/>
+<instance part="GND7" gate="1" x="185.42" y="71.12"/>
 </instances>
 <busses>
@@
 </segment>
 <segment>
-<wire x1="220.98" y1="157.48" x2="220.98" y2="160.02" width="0.1524" layer="91"/>
-<pinref part="C3" gate="G$1" pin="-"/>
-<pinref part="GND10" gate="1" pin="GND"/>
-</segment>
-<segment>
 <pinref part="BAT1" gate="G$1" pin="+"/>
 <pinref part="GND2" gate="1" pin="GND"/>
-<wire x1="180.34" y1="175.26" x2="182.88" y2="175.26" width="0.1524" layer="91"/>
+<wire x1="137.16" y1="165.1" x2="137.16" y2="175.26" width="0.1524" layer="91"/>
+<pinref part="C6" gate="G$1" pin="2"/>
+<wire x1="149.86" y1="167.64" x2="149.86" y2="165.1" width="0.1524" layer="91"/>
+<pinref part="IC1" gate="A1" pin="GND"/>
+<wire x1="149.86" y1="165.1" x2="165.1" y2="165.1" width="0.1524" layer="91"/>
+<wire x1="165.1" y1="165.1" x2="165.1" y2="167.64" width="0.1524" layer="91"/>
+<pinref part="C5" gate="G$1" pin="2"/>
+<wire x1="165.1" y1="165.1" x2="180.34" y2="165.1" width="0.1524" layer="91"/>
+<wire x1="180.34" y1="165.1" x2="180.34" y2="167.64" width="0.1524" layer="91"/>
+<junction x="165.1" y="165.1"/>
+<wire x1="137.16" y1="165.1" x2="149.86" y2="165.1" width="0.1524" layer="91"/>
+<junction x="137.16" y="165.1"/>
+<junction x="149.86" y="165.1"/>
 </segment>
 <segment>
@@
 <junction x="99.06" y="129.54"/>
 </segment>
+<segment>
+<pinref part="GND5" gate="1" pin="GND"/>
+<pinref part="U$6" gate="G$1" pin="P$1"/>
+<wire x1="12.7" y1="50.8" x2="17.78" y2="50.8" width="0.1524" layer="91"/>
+</segment>
+<segment>
+<pinref part="R1" gate="G$1" pin="2"/>
+<pinref part="GND6" gate="1" pin="GND"/>
+<wire x1="175.26" y1="76.2" x2="175.26" y2="73.66" width="0.1524" layer="91"/>
+</segment>
+<segment>
+<pinref part="R2" gate="G$1" pin="1"/>
+<pinref part="GND7" gate="1" pin="GND"/>
+<wire x1="185.42" y1="76.2" x2="185.42" y2="73.66" width="0.1524" layer="91"/>
+</segment>
 </net>
 <net name="EL_C" class="0">
-<segment>
-<wire x1="243.84" y1="129.54" x2="228.6" y2="129.54" width="0.1524" layer="91"/>
-<label x="236.22" y="129.54" size="1.778" layer="95"/>
-</segment>
 <segment>
 <wire x1="58.42" y1="132.08" x2="66.04" y2="132.08" width="0.1524" layer="91"/>
@@
 <pinref part="R3" gate="G$1" pin="2"/>
 </segment>
-</net>
-<net name="EL_D" class="0">
-<segment>
-<wire x1="243.84" y1="127" x2="228.6" y2="127" width="0.1524" layer="91"/>
-<label x="236.22" y="127" size="1.778" layer="95"/>
+<segment>
+<pinref part="IC2" gate="G$1" pin="RA4/T0CKI"/>
+<wire x1="119.38" y1="114.3" x2="109.22" y2="114.3" width="0.1524" layer="91"/>
+<label x="109.22" y="114.3" size="1.778" layer="91"/>
 </segment>
 </net>
@@
 <net name="VDD" class="0">
 <segment>
-<pinref part="BAT1" gate="G$1" pin="-"/>
 <pinref part="VDD1" gate="G$1" pin="VDD"/>
-<wire x1="233.68" y1="175.26" x2="220.98" y2="175.26" width="0.1524" layer="91"/>
-<wire x1="210.82" y1="175.26" x2="193.04" y2="175.26" width="0.1524" layer="91"/>
+<wire x1="233.68" y1="175.26" x2="210.82" y2="175.26" width="0.1524" layer="91"/>
 <pinref part="C2" gate="G$1" pin="1"/>
 <wire x1="210.82" y1="167.64" x2="210.82" y2="175.26" width="0.1524" layer="91"/>
-<pinref part="C3" gate="G$1" pin="+"/>
-<wire x1="210.82" y1="175.26" x2="220.98" y2="175.26" width="0.1524" layer="91"/>
-<wire x1="220.98" y1="175.26" x2="220.98" y2="167.64" width="0.1524" layer="91"/>
+<pinref part="IC1" gate="A1" pin="VO"/>
+<pinref part="C5" gate="G$1" pin="1"/>
+<wire x1="175.26" y1="175.26" x2="180.34" y2="175.26" width="0.1524" layer="91"/>
+<wire x1="180.34" y1="175.26" x2="198.12" y2="175.26" width="0.1524" layer="91"/>
+<junction x="180.34" y="175.26"/>
+<junction x="210.82" y="175.26"/>
+<pinref part="JP3" gate="G$1" pin="1"/>
+<wire x1="198.12" y1="175.26" x2="210.82" y2="175.26" width="0.1524" layer="91"/>
+<wire x1="198.12" y1="165.1" x2="198.12" y2="175.26" width="0.1524" layer="91"/>
+<junction x="198.12" y="175.26"/>
 </segment>
 <segment>
@@
 <label x="45.72" y="93.98" size="1.778" layer="91"/>
 </segment>
+<segment>
+<pinref part="IC2" gate="G$1" pin="INT0/AN4/RB0"/>
+<wire x1="177.8" y1="132.08" x2="187.96" y2="132.08" width="0.1524" layer="91"/>
+<label x="187.96" y="132.08" size="1.778" layer="91"/>
+</segment>
 </net>
 <net name="N$1" class="0">
@@
 </segment>
 </net>
+<net name="DEVICE_MAX_SET" class="0">
+<segment>
+<pinref part="U$6" gate="G$1" pin="P$2"/>
+<wire x1="43.18" y1="50.8" x2="58.42" y2="50.8" width="0.1524" layer="91"/>
+<label x="58.42" y="50.8" size="1.778" layer="91"/>
+</segment>
+<segment>
+<pinref part="IC2" gate="G$1" pin="INT2/P1B/RB2"/>
+<wire x1="177.8" y1="127" x2="187.96" y2="127" width="0.1524" layer="91"/>
+<label x="187.96" y="127" size="1.778" layer="91"/>
+</segment>
+</net>
+<net name="N$4" class="0">
+<segment>
+<pinref part="C6" gate="G$1" pin="1"/>
+<pinref part="IC1" gate="A1" pin="VI"/>
+<wire x1="149.86" y1="175.26" x2="154.94" y2="175.26" width="0.1524" layer="91"/>
+<pinref part="BAT1" gate="G$1" pin="-"/>
+<wire x1="147.32" y1="175.26" x2="149.86" y2="175.26" width="0.1524" layer="91"/>
+<junction x="149.86" y="175.26"/>
+</segment>
+</net>
+<net name="N$8" class="0">
+<segment>
+<pinref part="IC2" gate="G$1" pin="INT1/CK/TX/AN5/RB1"/>
+<wire x1="177.8" y1="129.54" x2="187.96" y2="129.54" width="0.1524" layer="91"/>
+<label x="187.96" y="129.54" size="1.778" layer="91"/>
+</segment>
+</net>
+<net name="NUM_LED" class="0">
+<segment>
+<pinref part="LED1" gate="G$1" pin="A"/>
+<wire x1="175.26" y1="93.98" x2="175.26" y2="99.06" width="0.1524" layer="91"/>
+<label x="170.18" y="99.06" size="1.778" layer="91"/>
+</segment>
+<segment>
+<pinref part="IC2" gate="G$1" pin="RA1/AN1/LVDIN"/>
+<wire x1="114.3" y1="121.92" x2="119.38" y2="121.92" width="0.1524" layer="91"/>
+<label x="109.22" y="121.92" size="1.778" layer="91"/>
+</segment>
+</net>
+<net name="MAX_LED" class="0">
+<segment>
+<pinref part="LED2" gate="G$1" pin="A"/>
+<wire x1="185.42" y1="93.98" x2="185.42" y2="99.06" width="0.1524" layer="91"/>
+<label x="185.42" y="99.06" size="1.778" layer="91"/>
+</segment>
+<segment>
+<pinref part="IC2" gate="G$1" pin="RA0/AN0"/>
+<wire x1="119.38" y1="124.46" x2="114.3" y2="124.46" width="0.1524" layer="91"/>
+<label x="109.22" y="124.46" size="1.778" layer="91"/>
+</segment>
+</net>

Commit message: v1.0 -- Fabbed Version
Parts:
- added LED3: (no value), led:LED3MM
- added R4: (no value), resistor:R-US_0204/5
- added U1: TRIAC, SparkFun:TRIACPTH
- IC1: value 7805L -> REG
Connections:
- removed net N$4: BAT1.-, C6.1, IC1.VI
- new net N$12: SV2.1, U1.M2
- new net N$13: SV2.3, U1.M1
- new net N$14: IC2.RA2/AN2/VREF-, U1.G
- new net N$7: IC2.RA3/AN3/VREF+, LED3.A
- new net N$9: BAT1.+, C6.1, IC1.VI
- net GND: now also BAT1.-, LED3.C; no longer BAT1.+
- net N$1: now also R4.1
- net N$8: now also JP4.1
- net VDD: now also R4.2
Other:
- moved on the sheet: BAT1, JP4, LED1
Changed lines of the file:
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@@
 <part name="C5" library="rcl" deviceset="C-US" device="025-025X050" value="1uF"/>
 <part name="C6" library="rcl" deviceset="C-US" device="025-025X050" value="1uF"/>
-<part name="IC1" library="linear" deviceset="78*" device="L" technology="05"/>
+<part name="IC1" library="linear" deviceset="78*" device="L" technology="05" value="REG"/>
 <part name="GND6" library="supply1" deviceset="GND" device=""/>
 <part name="GND7" library="supply1" deviceset="GND" device=""/>
+<part name="LED3" library="led" deviceset="LED" device="3MM"/>
+<part name="R4" library="resistor" deviceset="R-US_" device="0204/5"/>
+<part name="U1" library="SparkFun" deviceset="TRIAC" device="PTH" value="TRIAC"/>
 </parts>
 <sheets>
@@
 <instance part="U$5" gate="G$1" x="2.54" y="2.54"/>
 <instance part="J2" gate="G$1" x="104.14" y="81.28" rot="R270"/>
-<instance part="LED1" gate="G$1" x="175.26" y="91.44"/>
+<instance part="LED1" gate="G$1" x="175.26" y="93.98"/>
 <instance part="LED2" gate="G$1" x="185.42" y="91.44"/>
 <instance part="R1" gate="G$1" x="175.26" y="81.28" rot="R270"/>
 <instance part="R2" gate="G$1" x="185.42" y="81.28" rot="R90"/>
-<instance part="BAT1" gate="G$1" x="142.24" y="175.26"/>
+<instance part="BAT1" gate="G$1" x="137.16" y="175.26" rot="R180"/>
 <instance part="JP3" gate="G$1" x="198.12" y="162.56" rot="R270"/>
-<instance part="JP4" gate="G$1" x="93.98" y="170.18"/>
+<instance part="JP4" gate="G$1" x="215.9" y="129.54" rot="R180"/>
 <instance part="IC2" gate="G$1" x="149.86" y="124.46"/>
 <instance part="U$4" gate="G$1" x="27.94" y="106.68" rot="R270"/>
 <instance part="U$6" gate="G$1" x="22.86" y="50.8"/>
-<instance part="GND2" gate="1" x="137.16" y="162.56"/>
+<instance part="GND2" gate="1" x="137.16" y="160.02"/>
 <instance part="VDD1" gate="G$1" x="236.22" y="175.26" rot="R270"/>
 <instance part="Q1" gate="G$1" x="114.3" y="132.08" rot="R90"/>
@@
 <instance part="GND6" gate="1" x="175.26" y="71.12"/>
 <instance part="GND7" gate="1" x="185.42" y="71.12"/>
+<instance part="LED3" gate="G$1" x="93.98" y="116.84" rot="R270"/>
+<instance part="R4" gate="G$1" x="119.38" y="96.52"/>
+<instance part="U1" gate="G$1" x="226.06" y="81.28" smashed="yes">
+<attribute name="NAME" x="228.6" y="83.82" size="1.778" layer="95"/>
+<attribute name="VALUE" x="228.6" y="76.2" size="1.778" layer="96"/>
+</instance>
 </instances>
 <busses>
@@
 </segment>
 <segment>
-<pinref part="BAT1" gate="G$1" pin="+"/>
 <pinref part="GND2" gate="1" pin="GND"/>
-<wire x1="137.16" y1="165.1" x2="137.16" y2="175.26" width="0.1524" layer="91"/>
 <pinref part="C6" gate="G$1" pin="2"/>
 <wire x1="149.86" y1="167.64" x2="149.86" y2="165.1" width="0.1524" layer="91"/>
@@
 <wire x1="180.34" y1="165.1" x2="180.34" y2="167.64" width="0.1524" layer="91"/>
 <junction x="165.1" y="165.1"/>
-<wire x1="137.16" y1="165.1" x2="149.86" y2="165.1" width="0.1524" layer="91"/>
+<wire x1="137.16" y1="162.56" x2="149.86" y2="165.1" width="0.1524" layer="91"/>
+<junction x="149.86" y="165.1"/>
+<wire x1="121.92" y1="165.1" x2="124.46" y2="165.1" width="0.1524" layer="91"/>
+<wire x1="124.46" y1="165.1" x2="137.16" y2="165.1" width="0.1524" layer="91"/>
+<wire x1="137.16" y1="165.1" x2="137.16" y2="167.64" width="0.1524" layer="91"/>
+<pinref part="BAT1" gate="G$1" pin="-"/>
+<wire x1="132.08" y1="175.26" x2="124.46" y2="175.26" width="0.1524" layer="91"/>
+<wire x1="124.46" y1="175.26" x2="124.46" y2="165.1" width="0.1524" layer="91"/>
+<junction x="124.46" y="165.1"/>
+<wire x1="137.16" y1="162.56" x2="137.16" y2="165.1" width="0.1524" layer="91"/>
+<junction x="137.16" y="162.56"/>
 <junction x="137.16" y="165.1"/>
-<junction x="149.86" y="165.1"/>
 </segment>
 <segment>
@@
 <wire x1="99.06" y1="134.62" x2="99.06" y2="129.54" width="0.1524" layer="91"/>
 <junction x="99.06" y="129.54"/>
+<pinref part="LED3" gate="G$1" pin="C"/>
+<wire x1="88.9" y1="116.84" x2="86.36" y2="116.84" width="0.1524" layer="91"/>
+<wire x1="86.36" y1="116.84" x2="86.36" y2="127" width="0.1524" layer="91"/>
+<wire x1="86.36" y1="127" x2="99.06" y2="127" width="0.1524" layer="91"/>
+<junction x="99.06" y="127"/>
 </segment>
 <segment>
@@
 <label x="109.22" y="101.6" size="1.778" layer="91" rot="R90"/>
 </segment>
+<segment>
+<pinref part="R4" gate="G$1" pin="2"/>
+<wire x1="124.46" y1="96.52" x2="127" y2="96.52" width="0.1524" layer="91"/>
+<wire x1="127" y1="96.52" x2="127" y2="93.98" width="0.1524" layer="91"/>
+<label x="129.54" y="93.98" size="1.778" layer="91"/>
+</segment>
 </net>
 <net name="DEVICE_NUM_SET" class="0">
@@
 <segment>
 <pinref part="J2" gate="G$1" pin="VPP/MCLR"/>
-<wire x1="111.76" y1="93.98" x2="111.76" y2="111.76" width="0.1524" layer="91"/>
+<wire x1="111.76" y1="93.98" x2="111.76" y2="96.52" width="0.1524" layer="91"/>
 <pinref part="IC2" gate="G$1" pin="RA5/!MCLR"/>
+<wire x1="111.76" y1="96.52" x2="111.76" y2="111.76" width="0.1524" layer="91"/>
 <wire x1="111.76" y1="111.76" x2="119.38" y2="111.76" width="0.1524" layer="91"/>
+<pinref part="R4" gate="G$1" pin="1"/>
+<wire x1="114.3" y1="96.52" x2="111.76" y2="96.52" width="0.1524" layer="91"/>
+<junction x="111.76" y="96.52"/>
 </segment>
 </net>
@@
 <pinref part="LED1" gate="G$1" pin="C"/>
 <pinref part="R1" gate="G$1" pin="1"/>
+<wire x1="175.26" y1="88.9" x2="175.26" y2="86.36" width="0.1524" layer="91"/>
 </segment>
 </net>
@@
 </segment>
 </net>
-<net name="N$4" class="0">
-<segment>
-<pinref part="C6" gate="G$1" pin="1"/>
-<pinref part="IC1" gate="A1" pin="VI"/>
-<wire x1="149.86" y1="175.26" x2="154.94" y2="175.26" width="0.1524" layer="91"/>
-<pinref part="BAT1" gate="G$1" pin="-"/>
-<wire x1="147.32" y1="175.26" x2="149.86" y2="175.26" width="0.1524" layer="91"/>
-<junction x="149.86" y="175.26"/>
-</segment>
-</net>
 <net name="N$8" class="0">
 <segment>
 <pinref part="IC2" gate="G$1" pin="INT1/CK/TX/AN5/RB1"/>
-<wire x1="177.8" y1="129.54" x2="187.96" y2="129.54" width="0.1524" layer="91"/>
 <label x="187.96" y="129.54" size="1.778" layer="91"/>
+<wire x1="177.8" y1="129.54" x2="190.5" y2="129.54" width="0.1524" layer="91"/>
+<junction x="190.5" y="129.54"/>
+<wire x1="190.5" y1="129.54" x2="213.36" y2="129.54" width="0.1524" layer="91"/>
+<pinref part="JP4" gate="G$1" pin="1"/>
+<wire x1="213.36" y1="129.54" x2="215.9" y2="124.46" width="0.1524" layer="91"/>
+<wire x1="218.44" y1="129.54" x2="215.9" y2="124.46" width="0.1524" layer="91"/>
 </segment>
 </net>
@@
 <segment>
 <pinref part="LED1" gate="G$1" pin="A"/>
-<wire x1="175.26" y1="93.98" x2="175.26" y2="99.06" width="0.1524" layer="91"/>
+<wire x1="175.26" y1="96.52" x2="175.26" y2="99.06" width="0.1524" layer="91"/>
 <label x="170.18" y="99.06" size="1.778" layer="91"/>
 </segment>
@@
 </segment>
 </net>
+<net name="N$7" class="0">
+<segment>
+<pinref part="LED3" gate="G$1" pin="A"/>
+<pinref part="IC2" gate="G$1" pin="RA3/AN3/VREF+"/>
+<wire x1="96.52" y1="116.84" x2="119.38" y2="116.84" width="0.1524" layer="91"/>
+</segment>
+</net>
+<net name="N$9" class="0">
+<segment>
+<pinref part="BAT1" gate="G$1" pin="+"/>
+<pinref part="C6" gate="G$1" pin="1"/>
+<wire x1="142.24" y1="175.26" x2="149.86" y2="175.26" width="0.1524" layer="91"/>
+<pinref part="IC1" gate="A1" pin="VI"/>
+<wire x1="149.86" y1="175.26" x2="154.94" y2="175.26" width="0.1524" layer="91"/>
+<junction x="149.86" y="175.26"/>
+</segment>
+</net>
+<net name="N$12" class="0">
+<segment>
+<pinref part="SV2" gate="1" pin="1"/>
+<wire x1="213.36" y1="55.88" x2="220.98" y2="55.88" width="0.1524" layer="91"/>
+<wire x1="220.98" y1="55.88" x2="220.98" y2="86.36" width="0.1524" layer="91"/>
+<pinref part="U1" gate="G$1" pin="M2"/>
+<wire x1="220.98" y1="86.36" x2="226.06" y2="86.36" width="0.1524" layer="91"/>
+<wire x1="226.06" y1="86.36" x2="226.06" y2="83.82" width="0.1524" layer="91"/>
+</segment>
+</net>
+<net name="N$13" class="0">
+<segment>
+<pinref part="U1" gate="G$1" pin="M1"/>
+<wire x1="226.06" y1="76.2" x2="226.06" y2="60.96" width="0.1524" layer="91"/>
+<pinref part="SV2" gate="1" pin="3"/>
+<wire x1="226.06" y1="60.96" x2="213.36" y2="60.96" width="0.1524" layer="91"/>
+</segment>
+</net>
+<net name="N$14" class="0">
+<segment>
+<pinref part="U1" gate="G$1" pin="G"/>
+<wire x1="231.14" y1="78.74" x2="233.68" y2="78.74" width="0.1524" layer="91"/>
+<wire x1="233.68" y1="78.74" x2="233.68" y2="106.68" width="0.1524" layer="91"/>
+<wire x1="233.68" y1="106.68" x2="73.66" y2="106.68" width="0.1524" layer="91"/>
+<wire x1="73.66" y1="106.68" x2="73.66" y2="119.38" width="0.1524" layer="91"/>
+<pinref part="IC2" gate="G$1" pin="RA2/AN2/VREF-"/>
+<wire x1="73.66" y1="119.38" x2="119.38" y2="119.38" width="0.1524" layer="91"/>
+</segment>
+</net>
